Commit message: mpu6050

File: description/imu.xacro (robot description, xacro)
@@ -4,7 +4,4 @@
   <link name="imu_link">
     <visual name="imu_visual">
-      <geometry>
-        <mesh filename="package://bimo/meshes/MPU6050.dae"/>
-      </geometry>
     </visual>
   </link>
@@ -12,5 +9,5 @@
     <parent link="base_link"/>
     <child link="imu_link"/>
-    <origin xyz="0.190 0 0.10" rpy="0 0 0"/>
+    <origin xyz="0.150 0 0.08" rpy="0 0 0"/>
   </joint>
  <gazebo reference="imu_link">
